File: KiCad_Files/robi.kicad_pcb (KiCad board)
At the start: 2 copper layers, 53.7 x 59.6 mm, 8 parts, among them SW1 SW_DIP_x01

Commit message: added v1.2
Parts:
- D1, D2: footprint LED_THT:LED_D5.0mm -> blinkyparts:LED_D5.0mm_PLUS-Symbol
- moved D2 2.19 mm to (85.7, 51.8), turned to 90 degrees
- moved D1 2.03 mm to (69.3, 51.8), turned to 90 degrees
Routing:
- net VCC: track 62.7 -> 74.9 mm
- net GND: track 23.3 -> 21.6 mm
- net +3V0: track 21.5 -> 22.3 mm
Other:
- board text added: "-"
- board text added: "v1.2"
- board text removed: "v1.1"
