File: KiCad_Files/robi.kicad_sch (KiCad schematic)
At the start: 4 parts, among them SW1 SW_DIP_x01

Commit message: added v1.2
Parts:
- D1, D2: footprint LED_THT:LED_D5.0mm -> blinkyparts:LED_D5.0mm_PLUS-Symbol
Changed lines of the file:
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@@
       (effects (font (size 1.27 1.27)))
     )
-    (property "Footprint" "LED_THT:LED_D5.0mm" (at 121.92 62.23 0)
+    (property "Footprint" "blinkyparts:LED_D5.0mm_PLUS-Symbol" (at 121.92 62.23 0)
       (effects (font (size 1.27 1.27)) hide)
     )
@@
       (effects (font (size 1.27 1.27)))
     )
-    (property "Footprint" "LED_THT:LED_D5.0mm" (at 121.92 72.39 0)
+    (property "Footprint" "blinkyparts:LED_D5.0mm_PLUS-Symbol" (at 121.92 72.39 0)
       (effects (font (size 1.27 1.27)) hide)
     )
